Commit message: Complted Nav2 Stack, along with lots of other updates.

File: software/swarm_crawler/install/swarm_crawler/share/swarm_crawler/urdf/minibot.urdf (robot description, URDF)
Before this commit: robot minibot, 5 links, 4 joints
Links:
- removed link base_footprint
- removed link lidar_link
- added link camera_link, mass 0.114; collision cylinder length=0.18 radius=0.0508; visual cylinder length=0.18 radius=0.0508
- added link minibot_a_d435_link
- added link minibot_a_t265_pose_frame
- link base_link: geometry collision box size=${base_length} ${base_width} ${base_height}; visual box size=${base_length} ${base_width} ${base_height}
Joints:
- removed joint base_joint
- added joint d435_joint: type fixed, parent camera_link, child minibot_a_d435_link, origin xyz=0 0 0 rpy=0 0 0
- added joint extraneous_joint: type fixed, parent camera_link, child minibot_a_t265_pose_frame, origin xyz=0 0 0 rpy=0 0 0
- joint lidar_joint: child lidar_link -> camera_link; origin xyz=.6 0 0.13 rpy=0 0 0 -> xyz=.2 0 0.13 rpy=0 0 0

File: software/swarm_crawler/urdf/minibot.urdf (robot description, URDF)
Before this commit: robot minibot, 5 links, 4 joints
Links:
- removed link base_footprint
- added link minibot_a_d435_link
- added link minibot_a_t265_pose_frame
Joints:
- removed joint base_joint
- added joint d435_joint: type fixed, parent camera_link, child minibot_a_d435_link, origin xyz=0 0 0 rpy=0 0 0
- added joint extraneous_joint: type fixed, parent camera_link, child minibot_a_t265_pose_frame, origin xyz=0 0 0 rpy=0 0 0
- joint lidar_joint: origin xyz=.6 0 0.13 rpy=0 0 0 -> xyz=.2 0 0.13 rpy=0 0 0
