Commit message: updating before driver changes

File: software/swarm_crawler/urdf/minibot.urdf (robot description, URDF)
Before this commit: robot minibot, 5 links, 4 joints
Links:
- removed link lidar_link
- added link camera_link, mass 0.114; collision cylinder length=0.18 radius=0.0508; visual cylinder length=0.18 radius=0.0508
- link base_link: geometry collision box size=${base_length} ${base_width} ${base_height}; visual box size=${base_length} ${base_width} ${base_height}
Joints:
- joint lidar_joint: child lidar_link -> camera_link; origin xyz=0.215 0 0.13 rpy=0 0 0 -> xyz=.6 0 0.13 rpy=0 0 0

Commit message: Navigate to Aruco V1 Completed. Migrated back to ROS Galactic.

File: software/swarm_crawler/urdf/minibot.urdf (robot description, URDF)
Before this commit: robot minibot, 6 links, 5 joints
Joints:
- removed joint extraneous_joint
- added joint t265_joint: type fixed, parent camera_link, child minibot_a_t265_pose_frame, origin xyz=0.0 0.0 0.0 rpy=0 0 0
- joint d435_joint: origin xyz=0 0 0 rpy=0 0 0 -> xyz=0.0 0.0 0.0 rpy=0 0 0

Commit message: pre-merge changes

File: software/swarm_crawler/urdf/minibot.urdf (robot description, URDF)
Before this commit: robot minibot, 6 links, 5 joints
Links:
- removed link front_caster
- link base_link: geometry collision box size=${base_length} ${base_width} ${base_height}; visual mesh filename=package://swarm_crawler/meshes/minibot.stl scale=0.0015 0.0015 0.0015
- link camera_link: geometry collision cylinder length=0.05 radius=0.003; visual cylinder length=0.02 radius=0.0508
Joints:
- removed joint caster_joint
- removed joint lidar_joint
- added joint camera_joint: type fixed, parent base_link, child camera_link, origin xyz=${base_width/2} 0 ${base_length/2} rpy=0 0 0

Commit message: Adding changes that have been on the minibot. updated nav2 driving and other things.

File: software/swarm_crawler/urdf/minibot.urdf (robot description, URDF)
Before this commit: robot minibot, 5 links, 4 joints
Links:
- removed link minibot_a_t265_pose_frame
- link camera_link: mass 0.114 -> None
Joints:
- removed joint t265_joint
- joint camera_joint: origin xyz=${base_width/2} 0 ${base_length/2} rpy=0 0 0 -> xyz=.2 0 0 rpy=0 0 0
- joint imu_joint: origin xyz=-0.10 0 0.05 rpy=0 0 0 -> xyz=0 0 0.05 rpy=0 0 0
